File: plain60-b.kicad_pcb (KiCad board)
At the start: 2 copper layers, 284.7 x 94.2 mm, 175 parts, among them J1 USB_mini_micro_B, J2 ISP, K1 KEYSW, K10 KEYSW, K11 KEYSW, K12 KEYSW, K13 KEYSW, K14 KEYSW, K15 KEYSW, K15-1 KEYSW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

Commit message: Change website logo
Parts:
- G***: footprint Keeb_components:logo -> Keeb_components:logo_new
- moved G*** 5.98 mm to (26.8, 37.5)
- moved S1 0.68 mm to (25.6, 28.6)
Other:
- net class Default removed
- net class VCC removed
